File: kicad/ADV7513.sch (KiCad schematic (older format))
At the start: 44 parts, among them J1 HDMI, P1 5V, P2 SYNC, P3 I2C_INT, P4 AUDIO, P5 RED, P6 GREEN, P7 BLUE, U1 ADV7513, U2 NCP1117DT33G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

Commit message: cleaned up libraries
Parts:
- J1: symbol HDMI -> HDMI_conn
- P1: symbol CONN_01X02 -> Conn_01x02
- P2: symbol CONN_02X04 -> Conn_02x04_Top_Bottom
- P3: symbol CONN_01X04 -> Conn_01x04
- P4, P5, P6, P7: symbol CONN_02X08 -> Conn_02x08_Top_Bottom
- U2: symbol NCP1117DT33G -> NCP1117-3.3_TO252
- U3: symbol NCP1117DT18G -> NCP1117-1.8_TO252
Changed lines of the file:
@@
 EESchema Schematic File Version 2
-LIBS:ADV7513-rescue
 LIBS:power
 LIBS:device
@@
 LIBS:altera
 LIBS:HDMI
-LIBS:hdmi
 LIBS:ADV7513-cache
 EELAYER 25 0
@@
 $EndComp
 $Comp
-L NCP1117DT18G U3
+L NCP1117-1.8_TO252 U3
 U 1 1 58B1818F
 P 3150 1300
@@
 $EndComp
 $Comp
-L NCP1117DT33G U2
+L NCP1117-3.3_TO252 U2
 U 1 1 58B181E8
 P 1950 1300
@@
 $EndComp
 $Comp
-L CONN_01X02 P1
+L Conn_01x02 P1
 U 1 1 58B182DA
-P 700 1350
-F 0 "P1" H 700 1500 50  0000 C CNN
-F 1 "5V" V 800 1350 50  0000 C CNN
-F 2 "Pin_Headers:Pin_Header_Straight_1x02_Pitch2.54mm" H 700 1350 50  0001 C CNN
-F 3 "" H 700 1350 50  0000 C CNN
-	1    700  1350
+P 700 1400
+F 0 "P1" H 700 1550 50  0000 C CNN
+F 1 "5V" V 800 1400 50  0000 C CNN
+F 2 "Pin_Headers:Pin_Header_Straight_1x02_Pitch2.54mm" H 700 1400 50  0001 C CNN
+F 3 "" H 700 1400 50  0000 C CNN
+	1    700  1400
 	-1   0    0    1
 $EndComp
@@
 $EndComp
 $Comp
-L HDMI J1
+L HDMI_conn J1
 U 1 1 58B1F321
 P 9200 5100
@@
 Connection ~ 10250 1450
 $Comp
-L CONN_01X04 P3
+L Conn_01x04 P3
 U 1 1 58B60C9F
-P 800 7425
-F 0 "P3" H 800 7675 50  0000 C CNN
-F 1 "I2C_INT" V 900 7425 50  0000 C CNN
-F 2 "Pin_Headers:Pin_Header_Straight_1x04_Pitch2.54mm" H 800 7425 50  0001 C CNN
-F 3 "" H 800 7425 50  0000 C CNN
-	1    800  7425
+P 800 7475
+F 0 "P3" H 800 7725 50  0000 C CNN
+F 1 "I2C_INT" V 900 7475 50  0000 C CNN
+F 2 "Pin_Headers:Pin_Header_Straight_1x04_Pitch2.54mm" H 800 7475 50  0001 C CNN
+F 3 "" H 800 7475 50  0000 C CNN
+	1    800  7475
 	-1   0    0    1
 $EndComp
@@
 Connection ~ 1650 7575
 $Comp
-L CONN_02X08 P4
+L Conn_02x08_Top_Bottom P4
 U 1 1 58B64D3D
-P 1050 3375
-F 0 "P4" V 1050 3700 50  0000 C CNN
-F 1 "AUDIO" V 1050 3375 50  0000 C CNN
-F 2 "Pin_Headers:Pin_Header_Straight_2x08_Pitch2.54mm" H 1050 2175 50  0001 C CNN
-F 3 "" H 1050 2175 50  0000 C CNN
-	1    1050 3375
+P 1000 3325
+F 0 "P4" V 1050 3600 50  0000 C CNN
+F 1 "AUDIO" V 1050 3200 50  0000 C CNN
+F 2 "Pin_Headers:Pin_Header_Straight_2x08_Pitch2.54mm" H 1000 2125 50  0001 C CNN
+F 3 "" H 1000 2125 50  0000 C CNN
+	1    1000 3325
 	1    0    0    -1
 $EndComp
@@
 	1800 7475 1000 7475
 $Comp
-L CONN_02X08 P7
+L Conn_02x08_Top_Bottom P7
 U 1 1 58B5FF0F
-P 1050 6175
-F 0 "P7" V 1050 6500 50  0000 C CNN
-F 1 "BLUE" V 1050 6175 50  0000 C CNN
-F 2 "Pin_Headers:Pin_Header_Straight_2x08_Pitch2.54mm" H 1050 4975 50  0001 C CNN
-F 3 "" H 1050 4975 50  0000 C CNN
-	1    1050 6175
-	1    0    0    -1
-$EndComp
-$Comp
-L CONN_02X08 P6
+P 1000 6125
+F 0 "P7" V 1050 6400 50  0000 C CNN
+F 1 "BLUE" V 1050 6050 50  0000 C CNN
+F 2 "Pin_Headers:Pin_Header_Straight_2x08_Pitch2.54mm" H 1000 4925 50  0001 C CNN
+F 3 "" H 1000 4925 50  0000 C CNN
+	1    1000 6125
+	1    0    0    -1
+$EndComp
+$Comp
+L Conn_02x08_Top_Bottom P6
 U 1 1 58B5FFC7
-P 1050 5375
-F 0 "P6" V 1050 5700 50  0000 C CNN
-F 1 "GREEN" V 1050 5375 50  0000 C CNN
-F 2 "Pin_Headers:Pin_Header_Straight_2x08_Pitch2.54mm" H 1050 4175 50  0001 C CNN
-F 3 "" H 1050 4175 50  0000 C CNN
-	1    1050 5375
-	1    0    0    -1
-$EndComp
-$Comp
-L CONN_02X08 P5
+P 1000 5325
+F 0 "P6" V 1050 5600 50  0000 C CNN
+F 1 "GREEN" V 1050 5250 50  0000 C CNN
+F 2 "Pin_Headers:Pin_Header_Straight_2x08_Pitch2.54mm" H 1000 4125 50  0001 C CNN
+F 3 "" H 1000 4125 50  0000 C CNN
+	1    1000 5325
+	1    0    0    -1
+$EndComp
+$Comp
+L Conn_02x08_Top_Bottom P5
 U 1 1 58B6006C
-P 1050 4575
-F 0 "P5" V 1050 4900 50  0000 C CNN
-F 1 "RED" V 1050 4575 50  0000 C CNN
-F 2 "Pin_Headers:Pin_Header_Straight_2x08_Pitch2.54mm" H 1050 3375 50  0001 C CNN
-F 3 "" H 1050 3375 50  0000 C CNN
-	1    1050 4575
-	1    0    0    -1
-$EndComp
-$Comp
-L CONN_02X04 P2
+P 1000 4525
+F 0 "P5" V 1050 4800 50  0000 C CNN
+F 1 "RED" V 1050 4450 50  0000 C CNN
+F 2 "Pin_Headers:Pin_Header_Straight_2x08_Pitch2.54mm" H 1000 3325 50  0001 C CNN
+F 3 "" H 1000 3325 50  0000 C CNN
+	1    1000 4525
+	1    0    0    -1
+$EndComp
+$Comp
+L Conn_02x04_Top_Bottom P2
 U 1 1 58B600EE
-P 1050 3975
-F 0 "P2" V 1050 4100 50  0000 C CNN
-F 1 "SYNC" V 1050 3900 50  0000 C CNN
-F 2 "Pin_Headers:Pin_Header_Straight_2x04_Pitch2.54mm" H 1050 2775 50  0001 C CNN
-F 3 "" H 1050 2775 50  0000 C CNN
-	1    1050 3975
-	1    0    0    -1
-$EndComp
+P 1000 3925
+F 0 "P2" V 1050 4000 50  0000 C CNN
+F 1 "SYNC" V 1050 3800 50  0000 C CNN
+F 2 "Pin_Headers:Pin_Header_Straight_2x04_Pitch2.54mm" H 1000 2725 50  0001 C CNN
+F 3 "" H 1000 2725 50  0000 C CNN
+	1    1000 3925
+	1    0    0    -1
+$EndComp
